Commit message: Imported upstream version '0.0.2' of 'upstream'

File: urdf/robotont_realsense.urdf.xacro (robot description, xacro)
@@ -1,9 +1,8 @@
 <?xml version="1.0"?>
 <robot xmlns:xacro="http://ros.org/wiki/xacro" name="robotont">
-    <xacro:include filename="$(find realsense2_description)/urdf/_d435.urdf.xacro" />
+    <xacro:include filename="$(find realsense2_description)/urdf/_d435i.urdf.xacro" />
     <xacro:include filename="$(find robotont_description)/urdf/robotont_base.urdf.xacro"/>
     <xacro:arg name= "add_plug" default="false"/>
     <xacro:arg name= "simulated" default="false"/>
-    <xacro:property name= "prefix" value="$(arg prefix)"/>
     <!-- Camera assembly -->
     <link name="${prefix}camera_assembly_link1">
@@ -39,12 +38,12 @@
     <!-- Realsense -->
     <xacro:if value="$(arg simulated)">
-        <xacro:sensor_d435 parent="${prefix}base_link" use_nominal_extrinsics="true">
+        <xacro:sensor_d435i name="${prefix}camera" parent="${prefix}base_link" use_nominal_extrinsics="true">
             <origin xyz="-0.115 0 0.2025" rpy="0 0 0"/>
-        </xacro:sensor_d435>
+        </xacro:sensor_d435i>
     </xacro:if>
     <xacro:unless value="$(arg simulated)">
-        <xacro:sensor_d435 parent="${prefix}base_link" use_nominal_extrinsics="false">
+        <xacro:sensor_d435i name="${prefix}camera" parent="${prefix}base_link" use_nominal_extrinsics="false">
             <origin xyz="-0.115 0 0.2025" rpy="0 0 0"/>
-        </xacro:sensor_d435>
+        </xacro:sensor_d435i>
     </xacro:unless>
     <!-- Computer -->
